File: WRIST-PCB/WRIST.brd (EAGLE design)
At the start: 53 x 17.8 mm, 20 parts, among them Q3 BSS138, U3 LP5907-2.8V

Commit message: progress
Parts:
- added D10, D11, D4, D5, D6, D7, D8, D9: 1N4148, microbuilder:SOD-323
- added R10, R11, R12, R13, R14, R15, R16, R17, R18, R19, R20, R21, R22, R6, R8, R9: 10K, microbuilder:0603-NO
- moved J3 23.1 mm to (49.1, 11.7)
- moved J5 19.2 mm to (39.0, 11.8)
- moved J6 14.8 mm to (44.3, 11.7), turned to 270 degrees
- moved Q3 12.2 mm to (34.0, 9.91), turned to 0 degrees
- moved R7 11.1 mm to (28.8, 9.78)
- moved C4 9.48 mm to (23.7, 11.0)
- moved C5 9.43 mm to (23.7, 8.76)
- moved C6 7.13 mm to (18.7, 9.40), turned to 270 degrees
- moved U3 4.46 mm to (13.7, 9.27), turned to 270 degrees
- moved R3 1.92 mm to (8.76, 9.27)
- moved D2 0.51 mm to (5.97, 9.02)
- moved J2 0.40 mm to (3.43, 8.00)
- moved J1 0.38 mm to (2.41, 15.7)
Connections:
- removed net N$10: J4.12
- removed net N$11: J4.11
- removed net N$12: J4.10
- removed net N$13: J4.9
- removed net N$14: J4.8
- removed net N$15: J4.7
- removed net N$16: J4.6
- removed net N$17: J4.5
- removed net N$2: J4.20
- removed net N$22: J1.20
- removed net N$23: J1.19
- removed net N$24: J1.18
- removed net N$25: J1.17
- removed net N$26: J1.16
- removed net N$27: J1.15
- removed net N$28: J1.14
- removed net N$29: J1.13
- removed net N$3: J4.19
- removed net N$30: J1.12
- removed net N$31: J1.11
- removed net N$32: J1.10
- removed net N$33: J1.9
- removed net N$34: J1.8
- removed net N$35: J1.7
- removed net N$36: J1.6
- removed net N$37: J1.5
- removed net N$4: J4.18
- removed net N$5: J4.17
- removed net N$6: J4.16
- removed net N$7: J4.15
- removed net N$8: J4.14
- removed net N$9: J4.13
- new net GPIO_10: J1.20, J4.20, R20.1
- new net GPIO_3: J1.6, J4.6, R8.1
- new net GPIO_4: J1.8, J4.8, R10.1
- new net GPIO_5: J1.10, J4.10, R12.1
- new net GPIO_6: J1.12, J4.12, R14.1
- new net GPIO_7: J1.14, J4.14, R22.1
- new net GPIO_8: J1.16, J4.16, R16.1
- new net GPIO_9: J1.18, J4.18, R18.1
- new net XSHUT_10: D10.C, J1.19
- new net XSHUT_10_2.8V: D10.A, J4.19, R19.1
- new net XSHUT_3: D4.C, J1.5
- new net XSHUT_3_2.8V: D4.A, J4.5, R6.1
- new net XSHUT_4: D5.C, J1.7
- new net XSHUT_4_2.8V: D5.A, J4.7, R9.1
- new net XSHUT_5: D6.C, J1.9
- new net XSHUT_5_2.8V: D6.A, J4.9, R11.1
- new net XSHUT_6: D7.C, J1.11
- new net XSHUT_6_2.8V: D7.A, J4.11, R13.1
- new net XSHUT_7: D11.C, J1.13
- new net XSHUT_7_2.8V: D11.A, J4.13, R21.1
- new net XSHUT_8: D8.C, J1.15
- new net XSHUT_8_2.8V: D8.A, J4.15, R15.1
- new net XSHUT_9: D9.C, J1.17
- new net XSHUT_9_2.8V: D9.A, J4.17, R17.1
- net 2.8V: now also R10.2, R11.2, R12.2, R13.2, R14.2, R15.2, R16.2, R17.2, R18.2, R19.2, R20.2, R21.2, R22.2, R6.2, R8.2, R9.2
Routing:
- net 2.8V: track 3.05 -> 49.3 mm
- net XSHUT_9_2.8V: track 0.00 -> 4.45 mm
- net XSHUT_6_2.8V: track 0.00 -> 4.27 mm
- net XSHUT_4_2.8V: track 0.00 -> 4.27 mm
- net XSHUT_8_2.8V: track 0.00 -> 4.27 mm
- net XSHUT_3_2.8V: track 0.00 -> 4.27 mm
- net XSHUT_7_2.8V: track 0.00 -> 4.27 mm
- net XSHUT_5_2.8V: track 0.00 -> 4.27 mm
- net XSHUT_10_2.8V: track 0.00 -> 4.27 mm
- net GPIO_9: track 0.00 -> 2.20 mm
- net GPIO_8: track 0.00 -> 2.20 mm
- net GPIO_7: track 0.00 -> 2.20 mm
- net GPIO_6: track 0.00 -> 2.20 mm
- net GPIO_5: track 0.00 -> 2.20 mm
- net GPIO_4: track 0.00 -> 2.20 mm
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
Commit message: finish wrist pcb
Parts:
- moved J5 38.0 mm to (1.40, 6.60)
- moved C4 14.1 mm to (9.65, 11.6)
- moved J6 13.0 mm to (54.6, 3.68), turned to 90 degrees
- moved Q3 11.3 mm to (45.2, 11.8), turned to 180 degrees
- moved R7 9.61 mm to (38.1, 12.3)
- moved C5 9.12 mm to (32.4, 11.7)
- moved C6 7.91 mm to (26.2, 11.9)
- moved J1 7.24 mm to (4.32, 8.76)
- moved U3 7.00 mm to (20.2, 11.9)
- moved J3 6.19 mm to (54.6, 14.6)
- moved R3 6.19 mm to (14.4, 11.9)
- moved J2 3.06 mm to (1.40, 10.3)
- moved D2 2.65 mm to (5.21, 11.6), turned to 180 degrees
- moved D10 1.91 mm to (49.3, 5.33)
- moved D11 1.91 mm to (34.0, 5.33)
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Routing:
- net 2.8V: track 49.3 -> 106.7 mm, vias 0 -> 2
- net VCC: track 0.00 -> 49.8 mm, vias 0 -> 2
- net GND: track 0.00 -> 38.2 mm
- net SCL: track 0.00 -> 34.9 mm, vias 0 -> 3
- net SDA_3V: track 0.00 -> 32.7 mm, vias 0 -> 2
- net SCL_3V: track 0.00 -> 22.9 mm, vias 0 -> 2
- net SDA: track 0.00 -> 16.9 mm
- net N$1: track 0.00 -> 13.5 mm, vias 0 -> 2
- net GPIO_9: track 2.20 -> 9.06 mm
- net GPIO_8: track 2.20 -> 9.06 mm
- net GPIO_7: track 2.20 -> 9.06 mm
- net GPIO_6: track 2.20 -> 9.06 mm
- net GPIO_5: track 2.20 -> 9.06 mm
- net GPIO_4: track 2.20 -> 9.06 mm
- net GPIO_3: track 2.20 -> 9.06 mm
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Other:
- board size 53 x 17.8 mm -> 56.3 x 16.5 mm
