File: WRIST-PCB/WRIST.sch (EAGLE design)
At the start: 20 parts, among them Q3 BSS138, U3 LP5907-2.8V

Commit message: progress
Parts:
- added D10, D11, D4, D5, D6, D7, D8, D9: 1N4148, microbuilder:DIODESOD-323
- added R10, R11, R12, R13, R14, R15, R16, R17, R18, R19, R20, R21, R22, R6, R8, R9: 10K, microbuilder:RESISTOR_0603_NOOUT
Connections:
- removed net N$10: J4.12
- removed net N$11: J4.11
- removed net N$12: J4.10
- removed net N$13: J4.9
- removed net N$14: J4.8
- removed net N$15: J4.7
- removed net N$16: J4.6
- removed net N$17: J4.5
- removed net N$2: J4.20
- removed net N$22: J1.20
- removed net N$23: J1.19
- removed net N$24: J1.18
- removed net N$25: J1.17
- removed net N$26: J1.16
- removed net N$27: J1.15
- removed net N$28: J1.14
- removed net N$29: J1.13
- removed net N$3: J4.19
- removed net N$30: J1.12
- removed net N$31: J1.11
- removed net N$32: J1.10
- removed net N$33: J1.9
- removed net N$34: J1.8
- removed net N$35: J1.7
- removed net N$36: J1.6
- removed net N$37: J1.5
- removed net N$4: J4.18
- removed net N$5: J4.17
- removed net N$6: J4.16
- removed net N$7: J4.15
- removed net N$8: J4.14
- removed net N$9: J4.13
- new net GPIO_10: J1.20, J4.20, R20.1
- new net GPIO_3: J1.6, J4.6, R8.1
- new net GPIO_4: J1.8, J4.8, R10.1
- new net GPIO_5: J1.10, J4.10, R12.1
- new net GPIO_6: J1.12, J4.12, R14.1
- new net GPIO_7: J1.14, J4.14, R22.1
- new net GPIO_8: J1.16, J4.16, R16.1
- new net GPIO_9: J1.18, J4.18, R18.1
- new net XSHUT_10: D10.C, J1.19
- new net XSHUT_10_2.8V: D10.A, J4.19, R19.1
- new net XSHUT_3: D4.C, J1.5
- new net XSHUT_3_2.8V: D4.A, J4.5, R6.1
- new net XSHUT_4: D5.C, J1.7
- new net XSHUT_4_2.8V: D5.A, J4.7, R9.1
- new net XSHUT_5: D6.C, J1.9
- new net XSHUT_5_2.8V: D6.A, J4.9, R11.1
- new net XSHUT_6: D7.C, J1.11
- new net XSHUT_6_2.8V: D7.A, J4.11, R13.1
- new net XSHUT_7: D11.C, J1.13
- new net XSHUT_7_2.8V: D11.A, J4.13, R21.1
- new net XSHUT_8: D8.C, J1.15
- new net XSHUT_8_2.8V: D8.A, J4.15, R15.1
- new net XSHUT_9: D9.C, J1.17
- new net XSHUT_9_2.8V: D9.A, J4.17, R17.1
- net 2.8V: now also R10.2, R11.2, R12.2, R13.2, R14.2, R15.2, R16.2, R17.2, R18.2, R19.2, R20.2, R21.2, R22.2, R6.2, R8.2, R9.2
Other:
- moved on the sheet: J1, J3, J5
